Commit message: Use official KUKA KR6 R900-2 model

File: src/designgrounded_ros2/urdf/kr6_d405_workcell.urdf.xacro (robot description, xacro)
@@ -1,172 +1,13 @@
 <?xml version="1.0"?>
 <robot name="kr6_d405_workcell" xmlns:xacro="http://www.ros.org/wiki/xacro">
-  <material name="kuka_gray">
-    <color rgba="0.45 0.48 0.52 1.0"/>
-  </material>
-  <material name="kuka_dark">
-    <color rgba="0.10 0.11 0.13 1.0"/>
-  </material>
+  <xacro:include filename="$(find kuka_kr6_support)/urdf/kr6r900_2_macro.xacro"/>
+  <xacro:kuka_kr6r900_2 prefix=""/>
   <material name="d405_blue">
     <color rgba="0.12 0.48 0.78 1.0"/>
   </material>
-  <link name="base_link">
-    <visual>
-      <origin xyz="0 0 0.09" rpy="0 0 0"/>
-      <geometry><cylinder radius="0.10" length="0.18"/></geometry>
-      <material name="kuka_dark"/>
-    </visual>
-    <collision>
-      <origin xyz="0 0 0.09" rpy="0 0 0"/>
-      <geometry><cylinder radius="0.10" length="0.18"/></geometry>
-    </collision>
-    <inertial>
-      <origin xyz="0 0 0.09"/>
-      <mass value="8.0"/>
-      <inertia ixx="0.08" ixy="0" ixz="0" iyy="0.08" iyz="0" izz="0.08"/>
-    </inertial>
-  </link>
-  <joint name="joint_1" type="revolute">
-    <parent link="base_link"/>
-    <child link="link_1"/>
-    <origin xyz="0 0 0.18" rpy="0 0 0"/>
-    <axis xyz="0 0 1"/>
-    <limit lower="-3.14" upper="3.14" effort="100" velocity="1.5"/>
-    <dynamics damping="1.0" friction="0.1"/>
-  </joint>
-  <link name="link_1">
-    <visual>
-      <origin xyz="0 0 0.10"/>
-      <geometry><cylinder radius="0.08" length="0.20"/></geometry>
-      <material name="kuka_gray"/>
-    </visual>
-    <collision>
-      <origin xyz="0 0 0.10"/>
-      <geometry><cylinder radius="0.08" length="0.20"/></geometry>
-    </collision>
-    <inertial>
-      <origin xyz="0 0 0.10"/>
-      <mass value="5.0"/>
-      <inertia ixx="0.04" ixy="0" ixz="0" iyy="0.04" iyz="0" izz="0.03"/>
-    </inertial>
-  </link>
-  <joint name="joint_2" type="revolute">
-    <parent link="link_1"/>
-    <child link="link_2"/>
-    <origin xyz="0 0 0.20"/>
-    <axis xyz="0 1 0"/>
-    <limit lower="-2.35" upper="2.35" effort="100" velocity="1.5"/>
-  </joint>
-  <link name="link_2">
-    <visual>
-      <origin xyz="0 0 0.15"/>
-      <geometry><box size="0.09 0.08 0.30"/></geometry>
-      <material name="kuka_gray"/>
-    </visual>
-    <collision>
-      <origin xyz="0 0 0.15"/>
-      <geometry><box size="0.09 0.08 0.30"/></geometry>
-    </collision>
-    <inertial>
-      <origin xyz="0 0 0.15"/>
-      <mass value="4.5"/>
-      <inertia ixx="0.035" ixy="0" ixz="0" iyy="0.035" iyz="0" izz="0.01"/>
-    </inertial>
-  </link>
-  <joint name="joint_3" type="revolute">
-    <parent link="link_2"/>
-    <child link="link_3"/>
-    <origin xyz="0 0 0.30"/>
-    <axis xyz="0 1 0"/>
-    <limit lower="-2.60" upper="2.60" effort="80" velocity="1.8"/>
-  </joint>
-  <link name="link_3">
-    <visual>
-      <origin xyz="0 0 0.125"/>
-      <geometry><box size="0.075 0.07 0.25"/></geometry>
-      <material name="kuka_gray"/>
-    </visual>
-    <collision>
-      <origin xyz="0 0 0.125"/>
-      <geometry><box size="0.075 0.07 0.25"/></geometry>
-    </collision>
-    <inertial>
-      <origin xyz="0 0 0.125"/>
-      <mass value="3.2"/>
-      <inertia ixx="0.02" ixy="0" ixz="0" iyy="0.02" iyz="0" izz="0.008"/>
-    </inertial>
-  </link>
-  <joint name="joint_4" type="revolute">
-    <parent link="link_3"/>
-    <child link="link_4"/>
-    <origin xyz="0 0 0.25"/>
-    <axis xyz="1 0 0"/>
-    <limit lower="-3.14" upper="3.14" effort="40" velocity="2.0"/>
-  </joint>
-  <link name="link_4">
-    <visual>
-      <origin xyz="0 0 0.05"/>
-      <geometry><cylinder radius="0.045" length="0.10"/></geometry>
-      <material name="kuka_gray"/>
-    </visual>
-    <collision>
-      <origin xyz="0 0 0.05"/>
-      <geometry><cylinder radius="0.045" length="0.10"/></geometry>
-    </collision>
-    <inertial>
-      <origin xyz="0 0 0.05"/>
-      <mass value="1.4"/>
-      <inertia ixx="0.003" ixy="0" ixz="0" iyy="0.003" iyz="0" izz="0.002"/>
-    </inertial>
-  </link>
-  <joint name="joint_5" type="revolute">
-    <parent link="link_4"/>
-    <child link="link_5"/>
-    <origin xyz="0 0 0.10"/>
-    <axis xyz="0 1 0"/>
-    <limit lower="-2.60" upper="2.60" effort="30" velocity="2.2"/>
-  </joint>
-  <link name="link_5">
-    <visual>
-      <origin xyz="0 0 0.04"/>
-      <geometry><cylinder radius="0.04" length="0.08"/></geometry>
-      <material name="kuka_gray"/>
-    </visual>
-    <collision>
-      <origin xyz="0 0 0.04"/>
-      <geometry><cylinder radius="0.04" length="0.08"/></geometry>
-    </collision>
-    <inertial>
-      <origin xyz="0 0 0.04"/>
-      <mass value="0.9"/>
-      <inertia ixx="0.001" ixy="0" ixz="0" iyy="0.001" iyz="0" izz="0.0007"/>
-    </inertial>
-  </link>
-  <joint name="joint_6" type="revolute">
-    <parent link="link_5"/>
-    <child link="tool0"/>
-    <origin xyz="0 0 0.08"/>
-    <axis xyz="1 0 0"/>
-    <limit lower="-3.14" upper="3.14" effort="20" velocity="2.5"/>
-  </joint>
-  <link name="tool0">
-    <visual>
-      <origin xyz="0 0 0.03"/>
-      <geometry><cylinder radius="0.035" length="0.06"/></geometry>
-      <material name="kuka_dark"/>
-    </visual>
-    <collision>
-      <origin xyz="0 0 0.03"/>
-      <geometry><cylinder radius="0.035" length="0.06"/></geometry>
-    </collision>
-    <inertial>
-      <origin xyz="0 0 0.03"/>
-      <mass value="0.5"/>
-      <inertia ixx="0.0005" ixy="0" ixz="0" iyy="0.0005" iyz="0" izz="0.0003"/>
-    </inertial>
-  </link>
   <joint name="d405_joint" type="fixed">
     <parent link="tool0"/>
     <child link="d405_link"/>
-    <origin xyz="0.06 0 0.08" rpy="0 0 0"/>
+    <origin xyz="0 0 0.06" rpy="0 0 0"/>
   </joint>
   <link name="d405_link">
@@ -193,30 +34,30 @@
       <plugin>gazebo_ros2_control/GazeboSystem</plugin>
     </hardware>
-    <joint name="joint_1">
+    <joint name="joint_a1">
       <command_interface name="position"/>
       <state_interface name="position"/>
       <state_interface name="velocity"/>
     </joint>
-    <joint name="joint_2">
+    <joint name="joint_a2">
       <command_interface name="position"/>
       <state_interface name="position"/>
       <state_interface name="velocity"/>
     </joint>
-    <joint name="joint_3">
+    <joint name="joint_a3">
       <command_interface name="position"/>
       <state_interface name="position"/>
       <state_interface name="velocity"/>
     </joint>
-    <joint name="joint_4">
+    <joint name="joint_a4">
       <command_interface name="position"/>
       <state_interface name="position"/>
       <state_interface name="velocity"/>
     </joint>
-    <joint name="joint_5">
+    <joint name="joint_a5">
       <command_interface name="position"/>
       <state_interface name="position"/>
       <state_interface name="velocity"/>
     </joint>
-    <joint name="joint_6">
+    <joint name="joint_a6">
       <command_interface name="position"/>
       <state_interface name="position"/>
